Commit message: Add control for robot

File: description/robot_core.xacro (robot description, xacro)
@@ -34,4 +34,7 @@
     </xacro:inertial_box>
   </link>
+  <gazebo reference="chassis">
+    <material>Gazebo/White</material>
+  </gazebo>
   <joint name="chassis_joint" type="fixed">
     <parent link="base_link"/>
@@ -62,4 +65,7 @@
     </xacro:inertial_cylinder>
   </link>
+  <gazebo reference="left_wheel">
+    <material>Gazebo/Blue</material>
+  </gazebo>
   <!-- RIGHT WHEEL LINK-->
   <joint name="right_wheel_joint" type="continuous">
@@ -85,4 +91,7 @@
     </xacro:inertial_cylinder>
   </link>
+  <gazebo reference="right_wheel">
+    <material>Gazebo/Blue</material>
+  </gazebo>
   <!-- CASTER WHEEL LINK-->
   <joint name="caster_wheel_joint" type="fixed">
@@ -107,3 +116,8 @@
     </xacro:inertial_sphere>
   </link>
+  <gazebo reference="caster_wheel">
+    <material>Gazebo/Black</material>
+    <mu1 value="0.001"/>
+    <mu2 value="0.001"/>
+  </gazebo>
 </robot>
