Commit message: Add lidar simulation

File: description/gazebo_control.xacro (robot description, xacro)
@@ -3,9 +3,13 @@
     <gazebo>
         <plugin name="diff_drive" filename="libgazebo_ros_diff_drive.so">
+            <!-- Name of joint which Gazebo find in URDF file-->
             <left_joint>left_wheel_joint</left_joint>
             <right_joint>right_wheel_joint</right_joint>
+            <!-- Distance between 2 wheels with D = 0.1m-->
             <wheel_separation>0.35</wheel_separation>
             <wheel_diameter>0.1</wheel_diameter>
+            <!-- Max momen-->
             <max_wheel_torque>200</max_wheel_torque>
+            <!-- Max acceleration (gia toc)-->
             <max_wheel_acceleration>10.0</max_wheel_acceleration>
             <command_topic>cmd_vel</command_topic>

File: description/robot_core.xacro (robot description, xacro)
@@ -4,4 +4,7 @@
   <material name="white">
     <color rgba="1 1 1 1"/>
+  </material>
+    <material name="red">
+    <color rgba="1 0 0 1"/>
   </material>
   <material name="orange">
